File: Electronics/IDP Shield/IDP Shield.sch (EAGLE design)
At the start: 1 part, among them M1 IDP_PROTOBOARD

Commit message: Update schematics
Parts:
- added R10, R12: 560R, IDP_library:R-EU_0207/10
- added R11, R9: 56K, IDP_library:R-EU_0207/10
- added R2, R4: 10k, IDP_library:R-EU_0207/10
- added R3, R5: 220R, IDP_library:R-EU_0207/10
- added R6: 670R, IDP_library:R-EU_0207/10
- added R7, R8: 330R, IDP_library:R-EU_0207/10
- added SV1: LDR, IDP_library:FE02-1
- added SV2: LINE_SENS_1, IDP_library:FE04-1
- added SV3: LINE_SENS_2, IDP_library:FE04-1
- added SV4: LDR_LEDS, IDP_library:FE04-1
- added SV6: PHOTO_INT_1, IDP_library:FE04-1
- added SV7: ULTRASONIC_SENS, IDP_library:FE04-1
- added SV9: PHOTO_INT_2, IDP_library:FE04-1
Connections:
- new net BUTTON_GO: M1.D6
- new net COLOUR_SENS_BLUE: M1.D0, R7.1
- new net COLOUR_SENS_LDR: R6.1, SV1.1
- new net COLOUR_SENS_RED: M1.D1, R8.1
- new net LDR_SENS: M1.A2
- new net LED_AMBER: M1.A3
- new net LED_BLUE: M1.A4/SDA
- new net LED_RED: M1.A5/SCL
- new net LINE_SENS_1: M1.A0, R4.2, SV3.1
- new net LINE_SENS_2: M1.A1, R2.2, SV2.1
- new net N$1: R7.2, SV4.1
- new net N$11: R11.1, SV9.4
- new net N$2: R3.2, SV2.3
- new net N$3: R8.2, SV4.3
- new net N$4: R5.2, SV3.3
- new net N$6: M1.D7
- new net N$8: R9.1, SV6.4
- new net PHOTO_INT_1: M1.D4, R10.1, SV6.1
- new net PHOTO_INT_2: M1.D5, R12.1, SV9.1
- new net ULTRA_ECHO: M1.D3, SV7.2
- new net ULTRA_TRIG: M1.D2, SV7.3
- net +5V: now also R11.2, R2.1, R3.1, R4.1, R5.1, R6.2, R9.2, SV6.2, SV7.4, SV9.2
- net GND: now also R10.2, R12.2, SV1.2, SV2.2, SV2.4, SV3.2, SV3.4, SV4.2, SV4.4, SV6.3, SV7.1, SV9.3
